File: ZoumoBotRio.sch (KiCad schematic (older format))
At the start: 75 parts, among them CON1 BARREL_JACK, J1 Screw_Terminal_1x05, J2 Screw_Terminal_1x05, P1 USB_OTG, P10 Analog, P11 Digital, P12 Analog, P13 Digital, P2 Analog, P3 Digital, P4 Analog, P5 Digital, P6 Analog, P7 Digital, P8 Analog, P9 Digital, Q1 Q_PMOS_GDS, Q2 IR Receiver, Q3 IR Receiver, U1 ZLDO1117K50TC, U2 ATmega32U4-AU, Y1 16MHz

Commit message: Minor modifications to PCB, uploaded correct schematic
Parts:
- JP2: value PWR SW -> Power Switch
- Q1: value Q_PMOS_GDS -> 12v Regulator
Other:
- moved on the sheet: CON1, F1, JP2, Q1
